Commit message: new urdf

File: davie_ws/install/david_assembly_description/share/david_assembly_description/urdf/David_assembly.xacro (robot description, xacro)
@@ -1,7 +1,7 @@
 <?xml version="1.0" ?>
-<robot name="David_assembly" xmlns:xacro="http://www.ros.org/wiki/xacro">
-<xacro:include filename="$(find David_assembly_description)/urdf/materials.xacro" />
-<xacro:include filename="$(find David_assembly_description)/urdf/David_assembly.trans" />
-<xacro:include filename="$(find David_assembly_description)/urdf/David_assembly.gazebo" />
+<robot name="david_assembly" xmlns:xacro="http://www.ros.org/wiki/xacro">
+<xacro:include filename="$(find david_assembly_description)/urdf/materials.xacro" />
+<xacro:include filename="$(find david_assembly_description)/urdf/david_assembly.trans" />
+<xacro:include filename="$(find david_assembly_description)/urdf/david_assembly.gazebo" />
 <link name="base_link">
   <inertial>
@@ -13,5 +13,5 @@
     <origin xyz="0 0 0" rpy="0 0 0"/>
     <geometry>
-      <mesh filename="package://David_assembly_description/meshes/base_link.stl" scale="0.001 0.001 0.001"/>
+      <mesh filename="package://david_assembly_description/meshes/base_link.stl" scale="0.001 0.001 0.001"/>
     </geometry>
     <material name="silver"/>
@@ -20,5 +20,5 @@
     <origin xyz="0 0 0" rpy="0 0 0"/>
     <geometry>
-      <mesh filename="package://David_assembly_description/meshes/base_link.stl" scale="0.001 0.001 0.001"/>
+      <mesh filename="package://david_assembly_description/meshes/base_link.stl" scale="0.001 0.001 0.001"/>
     </geometry>
   </collision>
@@ -33,5 +33,5 @@
     <origin xyz="-0.107113 -0.009896 -0.03437" rpy="0 0 0"/>
     <geometry>
-      <mesh filename="package://David_assembly_description/meshes/Rotation_axis_1.stl" scale="0.001 0.001 0.001"/>
+      <mesh filename="package://david_assembly_description/meshes/Rotation_axis_1.stl" scale="0.001 0.001 0.001"/>
     </geometry>
     <material name="silver"/>
@@ -40,5 +40,5 @@
     <origin xyz="-0.107113 -0.009896 -0.03437" rpy="0 0 0"/>
     <geometry>
-      <mesh filename="package://David_assembly_description/meshes/Rotation_axis_1.stl" scale="0.001 0.001 0.001"/>
+      <mesh filename="package://david_assembly_description/meshes/Rotation_axis_1.stl" scale="0.001 0.001 0.001"/>
     </geometry>
   </collision>
@@ -53,5 +53,5 @@
     <origin xyz="0.029 -0.00986 -0.09145" rpy="0 0 0"/>
     <geometry>
-      <mesh filename="package://David_assembly_description/meshes/Arm1_1.stl" scale="0.001 0.001 0.001"/>
+      <mesh filename="package://david_assembly_description/meshes/Arm1_1.stl" scale="0.001 0.001 0.001"/>
     </geometry>
     <material name="silver"/>
@@ -60,5 +60,5 @@
     <origin xyz="0.029 -0.00986 -0.09145" rpy="0 0 0"/>
     <geometry>
-      <mesh filename="package://David_assembly_description/meshes/Arm1_1.stl" scale="0.001 0.001 0.001"/>
+      <mesh filename="package://david_assembly_description/meshes/Arm1_1.stl" scale="0.001 0.001 0.001"/>
     </geometry>
   </collision>
@@ -73,5 +73,5 @@
     <origin xyz="-0.041 -0.00986 -0.20331" rpy="0 0 0"/>
     <geometry>
-      <mesh filename="package://David_assembly_description/meshes/Arm2_1.stl" scale="0.001 0.001 0.001"/>
+      <mesh filename="package://david_assembly_description/meshes/Arm2_1.stl" scale="0.001 0.001 0.001"/>
     </geometry>
     <material name="silver"/>
@@ -80,5 +80,5 @@
     <origin xyz="-0.041 -0.00986 -0.20331" rpy="0 0 0"/>
     <geometry>
-      <mesh filename="package://David_assembly_description/meshes/Arm2_1.stl" scale="0.001 0.001 0.001"/>
+      <mesh filename="package://david_assembly_description/meshes/Arm2_1.stl" scale="0.001 0.001 0.001"/>
     </geometry>
   </collision>
@@ -93,5 +93,5 @@
     <origin xyz="0.029 -0.00986 -0.31517" rpy="0 0 0"/>
     <geometry>
-      <mesh filename="package://David_assembly_description/meshes/Arm3_1.stl" scale="0.001 0.001 0.001"/>
+      <mesh filename="package://david_assembly_description/meshes/Arm3_1.stl" scale="0.001 0.001 0.001"/>
     </geometry>
     <material name="silver"/>
@@ -100,5 +100,5 @@
     <origin xyz="0.029 -0.00986 -0.31517" rpy="0 0 0"/>
     <geometry>
-      <mesh filename="package://David_assembly_description/meshes/Arm3_1.stl" scale="0.001 0.001 0.001"/>
+      <mesh filename="package://david_assembly_description/meshes/Arm3_1.stl" scale="0.001 0.001 0.001"/>
     </geometry>
   </collision>
