Commit message: Cleanup

File: david_ws/src/urdf5_description/urdf/urdf5.xacro (robot description, xacro)
@@ -192,5 +192,6 @@
 </joint>
 <joint name="joint1" type="continuous">
-  <origin xyz="-0.0 -0.0 0.1662" rpy="0 0 0"/>
+  <!-- <origin xyz="-0.0 -0.0 0.1662" rpy="0 0 0"/> -->
+  <origin xyz="-0.0 -0.0 0.1662" rpy="0 0 3.141592653589793"/>
   <parent link="base_top_1"/>
   <child link="shaft_1"/>
